File: PCB/AHD-Switch.kicad_pcb (KiCad board)
At the start: 2 copper layers, 1.7 x 10.3 mm, 25 parts, among them J1 Conn_Coaxial, J2 Conn_Coaxial, J3 Conn_Coaxial, J4 Conn_01x02_Pin, J5 Conn_01x02_Pin, J6 Conn_01x02_Pin, K1 SRA-05VDC-CL, SW1 SW_Push, SW5 SW_Push, U1 TS5A63157DBV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

Commit message: Final PCB
Parts:
- removed K1: SRA-05VDC-CL, NightMeer:SRA-05VDC-CL
- added H1: MountingHole, MountingHole:MountingHole_3.2mm_M3, F.Cu at (99.2, 143.8)
- added H2: MountingHole, MountingHole:MountingHole_3.2mm_M3, F.Cu at (60.6, 105.9)
- added H3: MountingHole, MountingHole:MountingHole_3.2mm_M3, F.Cu at (60.6, 143.8)
- added R12: 1,2K, Resistor_THT:R_Axial_DIN0207_L6.3mm_D2.5mm_P10.16mm_Horizontal, F.Cu at (92.5, 109.3)
- added U5: CPC1017N, Package_SO:SOP-4_3.8x4.1mm_P2.54mm, F.Cu at (99.3, 107.8)
- R1, R2, R4: value 75R -> 75
- R10: value 1000R -> 3,9K
- R11, R3, R7, R8, R9: value R -> 10K
- R5, R6: value 68R -> 68
- U3: value PC817 -> CPC1017N; footprint Package_DIP:DIP-4_W7.62mm -> Package_SO:SOP-4_3.8x4.1mm_P2.54mm
- moved JP1 117.5 mm to (45.1, 144.0), turned to 90 degrees
- moved SW1 95.9 mm to (81.4, 143.7)
- moved R4 94.9 mm to (50.0, 144.0), turned to 90 degrees
- moved U2 91.2 mm to (74.8, 137.0), turned to 90 degrees
- moved R9 88.4 mm to (93.0, 131.9), turned to 90 degrees
- moved R8 87.9 mm to (88.3, 131.9), turned to 90 degrees
- moved R2 86.9 mm to (44.9, 128.8)
- moved U1 83.8 mm to (57.4, 116.0)
- moved R3 82.9 mm to (63.1, 122.7), turned to 90 degrees
- moved SW5 82.6 mm to (71.4, 143.7)
- moved J5 82.5 mm to (97.0, 82.7), turned to 180 degrees
- moved R11 76.0 mm to (83.6, 131.9), turned to 90 degrees
- moved R7 76.0 mm to (89.2, 108.9), turned to 180 degrees
- moved J3 74.0 mm to (31.0, 139.0), turned to 180 degrees
- moved R10 73.7 mm to (100.6, 89.1), turned to -90 degrees
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Connections:
- J3 pad 2: Net-(J3-Ext) -> GND
- JP1 pad 1: GND -> Net-(JP1-A)
- R4 pad 1: Net-(J3-Ext) -> Net-(JP1-A)
- U3 pad 1: Net-(R10-Pad2) -> Net-(R12-Pad2)
- U3 pad 3: D2 -> Radio-R
- U3 pad 4: +5V -> +12V
Routing:
- net +5V: track 0.00 -> 168.2 mm
- net +12V: track 0.00 -> 71.8 mm
- net Radio-R: track 0.00 -> 56.9 mm
- net D5: track 0.00 -> 51.7 mm
- net Net-(J3-In): track 0.00 -> 47.2 mm
- net GND: track 0.00 -> 29.7 mm, vias 0 -> 1
- net D6: track 0.00 -> 25.3 mm
- net D1: track 0.00 -> 24.4 mm
- net D2: track 0.00 -> 20.3 mm
- net D7: track 0.00 -> 20.2 mm
- net Net-(J1-In): track 0.00 -> 17.0 mm
- net Net-(J2-In): track 0.00 -> 16.9 mm
- net Signal-R: track 0.00 -> 6.86 mm
- net Net-(R6-Pad2): track 0.00 -> 5.92 mm
- net Net-(R10-Pad2): track 0.00 -> 5.80 mm
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- added copper zone on B.Cu, net GND
Other:
- board size 1.7 x 10.3 mm -> 72.9 x 69.8 mm
